Commit message: debug message from joy

File: real_rover/urdf/chassis.xacro (robot description, xacro)
@@ -194,5 +194,5 @@
   </xacro:macro>
   <xacro:wheel_joint
-    w_name="l_f"
+    w_name="left_forward"
     origin_y="${track/2}"
     origin_x="${wheelbase/2}"
@@ -202,5 +202,5 @@
     mu2="0.5"/>
   <xacro:wheel_joint
-    w_name="l_m"
+    w_name="left_middle"
     origin_y="${track/2}"
     origin_x="0"
@@ -210,5 +210,5 @@
     mu2="0.5"/>
   <xacro:wheel_joint
-    w_name="l_r"
+    w_name="left_rear"
     origin_y="${track/2}"
     origin_x="${-wheelbase/2}"
@@ -218,5 +218,5 @@
     mu2="0.5"/>
   <xacro:wheel_joint
-    w_name="r_f"
+    w_name="right_forward"
     origin_y="${-track/2}"
     origin_x="${wheelbase/2}"
@@ -226,5 +226,5 @@
     mu2="0.5"/>
   <xacro:wheel_joint
-    w_name="r_m"
+    w_name="right_middle"
     origin_y="${-track/2}"
     origin_x="0"
@@ -234,5 +234,5 @@
     mu2="0.5"/>
   <xacro:wheel_joint
-    w_name="r_r"
+    w_name="right_rear"
     origin_y="${-track/2}"
     origin_x="${-wheelbase/2}"

File: real_rover/urdf/ros2_control.xacro (robot description, xacro)
@@ -15,30 +15,30 @@
     </hardware>
     <!-- Конфигурация суставов -->
-    <joint name="base_to_l_f_wheel">
+    <joint name="base_to_left_forward_wheel">
       <state_interface name="velocity"/>
       <state_interface name="position"/>
       <command_interface name="velocity"/>
     </joint>
-    <joint name="base_to_l_m_wheel">
+    <joint name="base_to_left_middle_wheel">
       <state_interface name="velocity"/>
       <state_interface name="position"/>
       <command_interface name="velocity"/>
     </joint>
-    <joint name="base_to_l_r_wheel">
+    <joint name="base_to_left_rear_wheel">
       <state_interface name="velocity"/>
       <state_interface name="position"/>
       <command_interface name="velocity"/>
     </joint>
-    <joint name="base_to_r_f_wheel">
+    <joint name="base_to_right_forward_wheel">
       <state_interface name="velocity"/>
       <state_interface name="position"/>
       <command_interface name="velocity"/>
     </joint>
-    <joint name="base_to_r_m_wheel">
+    <joint name="base_to_right_middle_wheel">
       <state_interface name="velocity"/>
       <state_interface name="position"/>
       <command_interface name="velocity"/>
     </joint>
-    <joint name="base_to_r_r_wheel">
+    <joint name="base_to_right_rear_wheel">
       <state_interface name="velocity"/>
       <state_interface name="position"/>
