Commit message: worked odom

File: real_rover/urdf/ros2_control.xacro (robot description, xacro)
@@ -5,7 +5,7 @@
       <plugin>ros2_control_wheeled_robot_hardware/WheeledRobotHardware</plugin>
       <!-- Параметры UDP-соединения -->
-      <param name="udp_ip">127.0.0.1</param>  <!-- IP робота  192.168.3.106, для отладки 127.0.0.1 -->
-      <param name="udp_port">8889</param>         <!-- Порт робота 4001, для отладки 8889 -->
-      <param name="local_port">8888</param>       <!-- Локальный порт 4001,  для отладки 8888 -->
+      <param name="udp_ip">192.168.3.106</param>  <!-- IP робота  192.168.3.106, для отладки 127.0.0.1 -->
+      <param name="udp_port">4001</param>         <!-- Порт робота 4001, для отладки 8889 -->
+      <param name="local_port">4001</param>       <!-- Локальный порт 4001,  для отладки 8888 -->
       <!-- Параметры колес -->
       <param name="wheel_separation">0.8</param>  <!-- Расстояние между колесами (м) -->

File: rover_description/urdf/ros2_control.xacro (robot description, xacro)
@@ -1,47 +1,65 @@
 <?xml version="1.0"?>
-<robot xmlns:xacro="http://www.ros.org/wiki/xacro" name="trk211">
-  <!-- Конфигурация ros2_control для Gazebo -->
-  <ros2_control name="WheeledRobotSystem" type="system">
-    <hardware>
-      <plugin>gazebo_ros_control/GazeboWheeledRobotHardware</plugin>
-      <param name="wheel_separation">0.8</param>
-      <param name="wheel_radius">0.19</param>
-    </hardware>
-    <!-- Конфигурация суставов -->
-    <joint name="base_to_left_forward_wheel">
-      <state_interface name="velocity"/>
-      <state_interface name="position"/>
-      <command_interface name="velocity"/>
-    </joint>
-    <joint name="base_to_left_middle_wheel">
-      <state_interface name="velocity"/>
-      <state_interface name="position"/>
-      <command_interface name="velocity"/>
-    </joint>
-    <joint name="base_to_left_rear_wheel">
-      <state_interface name="velocity"/>
-      <state_interface name="position"/>
-      <command_interface name="velocity"/>
-    </joint>
-    <joint name="base_to_right_forward_wheel">
-      <state_interface name="velocity"/>
-      <state_interface name="position"/>
-      <command_interface name="velocity"/>
-    </joint>
-    <joint name="base_to_right_middle_wheel">
-      <state_interface name="velocity"/>
-      <state_interface name="position"/>
-      <command_interface name="velocity"/>
-    </joint>
-    <joint name="base_to_right_rear_wheel">
-      <state_interface name="velocity"/>
-      <state_interface name="position"/>
-      <command_interface name="velocity"/>
-    </joint>
-  </ros2_control>
-  <!-- Конфигурация Gazebo -->
-  <gazebo>
-    <plugin name="gazebo_ros_control" filename="libgazebo_ros_control.so">
-    </plugin>
-  </gazebo>
+<robot xmlns:xacro="http://www.ros.org/wiki/xacro">
+    <ros2_control name="GazeboSystem" type="system">
+        <hardware>
+            <plugin>gazebo_ros2_control/GazeboSystem</plugin>
+        </hardware>
+        <joint name="base_to_l_f_wheel">
+            <command_interface name="velocity">
+                <param name="min">-10</param>
+                <param name="max">10</param>
+            </command_interface>
+            <state_interface name="velocity"/>
+            <state_interface name="position"/>
+        </joint>
+        <joint name="base_to_l_m_wheel">
+            <command_interface name="velocity">
+                <param name="min">-10</param>
+                <param name="max">10</param>
+            </command_interface>
+            <state_interface name="velocity"/>
+            <state_interface name="position"/>
+        </joint>
+        <joint name="base_to_l_r_wheel">
+            <command_interface name="velocity">
+                <param name="min">-10</param>
+                <param name="max">10</param>
+            </command_interface>
+            <state_interface name="velocity"/>
+            <state_interface name="position"/>
+        </joint>
+        <joint name="base_to_r_f_wheel">
+            <command_interface name="velocity">
+                <param name="min">-10</param>
+                <param name="max">10</param>
+            </command_interface>
+            <state_interface name="velocity"/>
+            <state_interface name="position"/>
+        </joint>
+        <joint name="base_to_r_m_wheel">
+            <command_interface name="velocity">
+                <param name="min">-10</param>
+                <param name="max">10</param>
+            </command_interface>
+            <state_interface name="velocity"/>
+            <state_interface name="position"/>
+        </joint>
+        <joint name="base_to_r_r_wheel">
+            <command_interface name="velocity">
+                <param name="min">-10</param>
+                <param name="max">10</param>
+            </command_interface>
+            <state_interface name="velocity"/>
+            <state_interface name="position"/>
+        </joint>
+    </ros2_control>
+    <gazebo>
+        <plugin name="gazebo_ros2_control" filename="libgazebo_ros2_control.so">
+            <parameters>$(find rover_description)/config/my_controllers.yaml</parameters>
+        </plugin>
+        <updateRate>30</updateRate>
+ <!--   <ros>
+          <remapping>odom:=odom/unfiltered</remapping>
+        </ros> -->
+    </gazebo>
 </robot>
