Commit message: unfixed ekf rotation, fixed odom & velodyne filter dropping message

File: rover_description/urdf/imu.xacro (robot description, xacro)
@@ -39,5 +39,5 @@
       <pose relative_to='xsens_link'>0 0 0 0 0 0</pose>
       <always_on>true</always_on>
-      <update_rate>100</update_rate>
+      <update_rate>5</update_rate>
       <!--reduced version of the plugin for ros2 without params-->
       <plugin filename="libgazebo_ros_imu_sensor.so" name="imu_plugin">

File: rover_description/urdf/ros2_control.xacro (robot description, xacro)
@@ -8,30 +8,48 @@
     <!-- Конфигурация суставов -->
     <joint name="base_to_l_f_wheel">
-      <command_interface name="velocity"/>
+      <command_interface name="velocity">
+        <param name="min">-10</param>
+        <param name="max">10</param>
+      </command_interface>
       <state_interface name="velocity"/>
       <state_interface name="position"/>
     </joint>
     <joint name="base_to_l_m_wheel">
-      <command_interface name="velocity"/>
+      <command_interface name="velocity">
+        <param name="min">-10</param>
+        <param name="max">10</param>
+      </command_interface>
       <state_interface name="velocity"/>
       <state_interface name="position"/>
     </joint>
     <joint name="base_to_l_r_wheel">
-      <command_interface name="velocity"/>
+      <command_interface name="velocity">
+        <param name="min">-10</param>
+        <param name="max">10</param>
+      </command_interface>
       <state_interface name="velocity"/>
       <state_interface name="position"/>
     </joint>
     <joint name="base_to_r_f_wheel">
-      <command_interface name="velocity"/>
+      <command_interface name="velocity">
+        <param name="min">-10</param>
+        <param name="max">10</param>
+      </command_interface>
       <state_interface name="velocity"/>
       <state_interface name="position"/>
     </joint>
     <joint name="base_to_r_m_wheel">
-      <command_interface name="velocity"/>
+      <command_interface name="velocity">
+        <param name="min">-5</param>
+        <param name="max">5</param>
+      </command_interface>
       <state_interface name="velocity"/>
       <state_interface name="position"/>
     </joint>
     <joint name="base_to_r_r_wheel">
-      <command_interface name="velocity"/>
+      <command_interface name="velocity">
+        <param name="min">-10</param>
+        <param name="max">10</param>
+      </command_interface>
       <state_interface name="velocity"/>
       <state_interface name="position"/>
@@ -39,8 +57,12 @@
   </ros2_control>
   <!-- Плагин Gazebo для ros2_control -->
-  <gazebo>
-    <plugin name="gazebo_ros2_control" filename="libgazebo_ros2_control.so">
-      <parameters>$(find rover_description)/config/my_controllers.yaml</parameters>
-    </plugin>
-  </gazebo>
+    <gazebo>
+        <plugin name="gazebo_ros2_control" filename="libgazebo_ros2_control.so">
+            <parameters>$(find rover_description)/config/my_controllers.yaml</parameters>
+        </plugin>
+        <updateRate>20</updateRate>
+ <!--   <ros>
+          <remapping>odom:=odom/unfiltered</remapping>
+        </ros> -->
+    </gazebo>
 </robot>

File: velodyne_simulator/velodyne_description/urdf/VLP-16.urdf.xacro (robot description, xacro)
@@ -2,5 +2,5 @@
 <robot xmlns:xacro="http://www.ros.org/wiki/xacro" name="VLP-16">
   <xacro:property name="M_PI" value="3.1415926535897931" />
-  <xacro:macro name="VLP-16" params="*origin parent:=base_link name:=velodyne tf_prefix:='' topic:=/velodyne_points organize_cloud:=false hz:=5 lasers:=16 samples:=1875 collision_range:=0.3 min_range:=0.9 max_range:=30.0 noise:=0.008 min_angle:=-${M_PI} max_angle:=${M_PI} gpu:=false">
+  <xacro:macro name="VLP-16" params="*origin parent:=base_link name:=velodyne tf_prefix:='' topic:=/velodyne_points organize_cloud:=false hz:=10 lasers:=16 samples:=1875 collision_range:=0.3 min_range:=0.9 max_range:=30.0 noise:=0.008 min_angle:=-${M_PI} max_angle:=${M_PI} gpu:=false">
     <joint name="${name}_base_mount_joint" type="fixed">
       <xacro:insert_block name="origin" />

Commit message: nav2 trouble

File: rover_description/urdf/imu.xacro (robot description, xacro)
@@ -39,5 +39,5 @@
       <pose relative_to='xsens_link'>0 0 0 0 0 0</pose>
       <always_on>true</always_on>
-      <update_rate>5</update_rate>
+      <update_rate>100</update_rate>
       <!--reduced version of the plugin for ros2 without params-->
       <plugin filename="libgazebo_ros_imu_sensor.so" name="imu_plugin">

File: rover_description/urdf/ros2_control.xacro (robot description, xacro)
@@ -1,39 +1,68 @@
 <?xml version="1.0"?>
-<robot xmlns:xacro="http://www.ros.org/wiki/xacro">
+<robot xmlns:xacro="http://www.ros.org/wiki/xacro" name="trk211">
+  <!-- Конфигурация ros2_control -->
+  <ros2_control name="GazeboSystem" type="system">
+    <hardware>
+      <plugin>gazebo_ros2_control/GazeboSystem</plugin>
+    </hardware>
+    <!-- Конфигурация суставов -->
+    <joint name="base_to_l_f_wheel">
+      <command_interface name="velocity">
+        <param name="min">-10</param>
+        <param name="max">10</param>
+      </command_interface>
+      <state_interface name="velocity"/>
+      <state_interface name="position"/>
+    </joint>
+    <joint name="base_to_l_m_wheel">
+      <command_interface name="velocity">
+        <param name="min">-10</param>
+        <param name="max">10</param>
+      </command_interface>
+      <state_interface name="velocity"/>
+      <state_interface name="position"/>
+    </joint>
+    <joint name="base_to_l_r_wheel">
+      <command_interface name="velocity">
+        <param name="min">-10</param>
+        <param name="max">10</param>
+      </command_interface>
+      <state_interface name="velocity"/>
+      <state_interface name="position"/>
+    </joint>
+    <joint name="base_to_r_f_wheel">
+      <command_interface name="velocity">
+        <param name="min">-10</param>
+        <param name="max">10</param>
+      </command_interface>
+      <state_interface name="velocity"/>
+      <state_interface name="position"/>
+    </joint>
+    <joint name="base_to_r_m_wheel">
+      <command_interface name="velocity">
+        <param name="min">-5</param>
+        <param name="max">5</param>
+      </command_interface>
+      <state_interface name="velocity"/>
+      <state_interface name="position"/>
+    </joint>
+    <joint name="base_to_r_r_wheel">
+      <command_interface name="velocity">
+        <param name="min">-10</param>
+        <param name="max">10</param>
+      </command_interface>
+      <state_interface name="velocity"/>
+      <state_interface name="position"/>
+    </joint>
+  </ros2_control>
+  <!-- Плагин Gazebo для ros2_control -->
     <gazebo>
-        <plugin name="diff_drive" filename="libgazebo_ros_diff_drive.so">
-            <!-- Wheel Information -->
-            <num_wheel_pairs>3</num_wheel_pairs>
-            <left_joint>base_to_l_f_wheel</left_joint>
-            <left_joint>base_to_l_m_wheel</left_joint>
-            <left_joint>base_to_l_r_wheel</left_joint>
-            <right_joint>base_to_r_f_wheel</right_joint>
-            <right_joint>base_to_r_m_wheel</right_joint>
-            <right_joint>base_to_r_r_wheel</right_joint>
-            <wheel_separation>0.8</wheel_separation>
-            <wheel_diameter>0.38</wheel_diameter>
-            <!-- Limits -->
-            <max_wheel_torque>200</max_wheel_torque>
-            <max_wheel_acceleration>10.0</max_wheel_acceleration>
-            <!-- Output -->
-            <odometry_topic>odom</odometry_topic>
-            <odometry_frame>odom</odometry_frame>
-            <robot_base_frame>root_link</robot_base_frame>
-            <publish_odom>true</publish_odom>
-            <publish_odom_tf>true</publish_odom_tf>
-            <publish_wheel_tf>true</publish_wheel_tf>
+        <plugin name="gazebo_ros2_control" filename="libgazebo_ros2_control.so">
+            <parameters>$(find rover_description)/config/my_controllers.yaml</parameters>
         </plugin>
-        <!--plugin name="joint_state" filename="libgazebo_ros_joint_state_publisher.so">
-            <ros>
-                <remapping>~/out:=joint_states</remapping>
-            </ros>
-            <update_rate>30</update_rate>
-            <joint_name>base_to_l_f_wheel</joint_name>
-            <joint_name>base_to_l_m_wheel</joint_name>
-            <joint_name>base_to_l_r_wheel</joint_name>
-            <joint_name>base_to_r_f_wheel</joint_name>
-            <joint_name>base_to_r_m_wheel</joint_name>
-            <joint_name>base_to_r_r_wheel</joint_name>
-        </plugin-->
+        <updateRate>20</updateRate>
+ <!--   <ros>
+          <remapping>odom:=odom/unfiltered</remapping>
+        </ros> -->
     </gazebo>
 </robot>

File: rover_description/urdf/trk211.xacro (robot description, xacro)
@@ -3,5 +3,5 @@
   <!-- Включение файлов -->
   <xacro:include filename="chassis.xacro"/>
-  <xacro:include filename="ros2_control.xacro"/>
+  <xacro:include filename="gazebo_control.xacro"/>
   <xacro:include filename="imu.xacro"/>
   <xacro:include filename="$(find velodyne_description)/urdf/VLP-16.urdf.xacro"/>
@@ -14,5 +14,7 @@
   <xacro:include filename="$(find realsense2_description)/urdf/_d415.urdf.xacro"/>
   <xacro:include filename="depth_camera.xacro"/>
-  <xacro:include filename="gazebo_control.xacro"/>-->
+  <xacro:include filename="gazebo_control.xacro"/>
+  <xacro:include filename="ros2_control.xacro"/>
+  -->
   <!--xacro:include filename="camera.xacro"/-->
 </robot>
