Commit message: low obstacles detecting, odom fix required

File: rover_description/urdf/ros2_control.xacro (robot description, xacro)
@@ -1,68 +1,39 @@
 <?xml version="1.0"?>
-<robot xmlns:xacro="http://www.ros.org/wiki/xacro" name="trk211">
-  <!-- Конфигурация ros2_control -->
-  <ros2_control name="GazeboSystem" type="system">
-    <hardware>
-      <plugin>gazebo_ros2_control/GazeboSystem</plugin>
-    </hardware>
-    <!-- Конфигурация суставов -->
-    <joint name="base_to_l_f_wheel">
-      <command_interface name="velocity">
-        <param name="min">-10</param>
-        <param name="max">10</param>
-      </command_interface>
-      <state_interface name="velocity"/>
-      <state_interface name="position"/>
-    </joint>
-    <joint name="base_to_l_m_wheel">
-      <command_interface name="velocity">
-        <param name="min">-10</param>
-        <param name="max">10</param>
-      </command_interface>
-      <state_interface name="velocity"/>
-      <state_interface name="position"/>
-    </joint>
-    <joint name="base_to_l_r_wheel">
-      <command_interface name="velocity">
-        <param name="min">-10</param>
-        <param name="max">10</param>
-      </command_interface>
-      <state_interface name="velocity"/>
-      <state_interface name="position"/>
-    </joint>
-    <joint name="base_to_r_f_wheel">
-      <command_interface name="velocity">
-        <param name="min">-10</param>
-        <param name="max">10</param>
-      </command_interface>
-      <state_interface name="velocity"/>
-      <state_interface name="position"/>
-    </joint>
-    <joint name="base_to_r_m_wheel">
-      <command_interface name="velocity">
-        <param name="min">-5</param>
-        <param name="max">5</param>
-      </command_interface>
-      <state_interface name="velocity"/>
-      <state_interface name="position"/>
-    </joint>
-    <joint name="base_to_r_r_wheel">
-      <command_interface name="velocity">
-        <param name="min">-10</param>
-        <param name="max">10</param>
-      </command_interface>
-      <state_interface name="velocity"/>
-      <state_interface name="position"/>
-    </joint>
-  </ros2_control>
-  <!-- Плагин Gazebo для ros2_control -->
+<robot xmlns:xacro="http://www.ros.org/wiki/xacro">
     <gazebo>
-        <plugin name="gazebo_ros2_control" filename="libgazebo_ros2_control.so">
-            <parameters>$(find rover_description)/config/my_controllers.yaml</parameters>
+        <plugin name="diff_drive" filename="libgazebo_ros_diff_drive.so">
+            <!-- Wheel Information -->
+            <num_wheel_pairs>3</num_wheel_pairs>
+            <left_joint>base_to_l_f_wheel</left_joint>
+            <left_joint>base_to_l_m_wheel</left_joint>
+            <left_joint>base_to_l_r_wheel</left_joint>
+            <right_joint>base_to_r_f_wheel</right_joint>
+            <right_joint>base_to_r_m_wheel</right_joint>
+            <right_joint>base_to_r_r_wheel</right_joint>
+            <wheel_separation>0.8</wheel_separation>
+            <wheel_diameter>0.38</wheel_diameter>
+            <!-- Limits -->
+            <max_wheel_torque>200</max_wheel_torque>
+            <max_wheel_acceleration>10.0</max_wheel_acceleration>
+            <!-- Output -->
+            <odometry_topic>odom</odometry_topic>
+            <odometry_frame>odom</odometry_frame>
+            <robot_base_frame>root_link</robot_base_frame>
+            <publish_odom>true</publish_odom>
+            <publish_odom_tf>true</publish_odom_tf>
+            <publish_wheel_tf>true</publish_wheel_tf>
         </plugin>
-        <updateRate>20</updateRate>
- <!--   <ros>
-          <remapping>odom:=odom/unfiltered</remapping>
-        </ros> -->
+        <!--plugin name="joint_state" filename="libgazebo_ros_joint_state_publisher.so">
+            <ros>
+                <remapping>~/out:=joint_states</remapping>
+            </ros>
+            <update_rate>30</update_rate>
+            <joint_name>base_to_l_f_wheel</joint_name>
+            <joint_name>base_to_l_m_wheel</joint_name>
+            <joint_name>base_to_l_r_wheel</joint_name>
+            <joint_name>base_to_r_f_wheel</joint_name>
+            <joint_name>base_to_r_m_wheel</joint_name>
+            <joint_name>base_to_r_r_wheel</joint_name>
+        </plugin-->
     </gazebo>
 </robot>

Commit message: shit

File: rover_description/urdf/ros2_control.xacro (robot description, xacro)
@@ -1,65 +1,62 @@
 <?xml version="1.0"?>
-<robot xmlns:xacro="http://www.ros.org/wiki/xacro" name="trk211">
-  <!-- Конфигурация ros2_control -->
-  <ros2_control name="GazeboSystem" type="system">
-    <hardware>
-      <plugin>gazebo_ros2_control/GazeboSystem</plugin>
-    </hardware>
-    <!-- Конфигурация суставов -->
-    <joint name="base_to_l_f_wheel">
-      <command_interface name="velocity">
-        <param name="min">-10</param>
-        <param name="max">10</param>
-      </command_interface>
-      <state_interface name="velocity"/>
-      <state_interface name="position"/>
-    </joint>
-    <joint name="base_to_l_m_wheel">
-      <command_interface name="velocity">
-        <param name="min">-10</param>
-        <param name="max">10</param>
-      </command_interface>
-      <state_interface name="velocity"/>
-      <state_interface name="position"/>
-    </joint>
-    <joint name="base_to_l_r_wheel">
-      <command_interface name="velocity">
-        <param name="min">-10</param>
-        <param name="max">10</param>
-      </command_interface>
-      <state_interface name="velocity"/>
-      <state_interface name="position"/>
-    </joint>
-    <joint name="base_to_r_f_wheel">
-      <command_interface name="velocity">
-        <param name="min">-10</param>
-        <param name="max">10</param>
-      </command_interface>
-      <state_interface name="velocity"/>
-      <state_interface name="position"/>
-    </joint>
-    <joint name="base_to_r_m_wheel">
-      <command_interface name="velocity">
-        <param name="min">-5</param>
-        <param name="max">5</param>
-      </command_interface>
-      <state_interface name="velocity"/>
-      <state_interface name="position"/>
-    </joint>
-    <joint name="base_to_r_r_wheel">
-      <command_interface name="velocity">
-        <param name="min">-10</param>
-        <param name="max">10</param>
-      </command_interface>
-      <state_interface name="velocity"/>
-      <state_interface name="position"/>
-    </joint>
-  </ros2_control>
-  <!-- Плагин Gazebo для ros2_control -->
+<robot xmlns:xacro="http://www.ros.org/wiki/xacro">
+    <ros2_control name="GazeboSystem" type="system">
+        <hardware>
+            <plugin>gazebo_ros2_control/GazeboSystem</plugin>
+        </hardware>
+        <joint name="base_to_l_f_wheel">
+            <command_interface name="velocity">
+                <param name="min">-10</param>
+                <param name="max">10</param>
+            </command_interface>
+            <state_interface name="velocity"/>
+            <state_interface name="position"/>
+        </joint>
+        <joint name="base_to_l_m_wheel">
+            <command_interface name="velocity">
+                <param name="min">-10</param>
+                <param name="max">10</param>
+            </command_interface>
+            <state_interface name="velocity"/>
+            <state_interface name="position"/>
+        </joint>
+        <joint name="base_to_l_r_wheel">
+            <command_interface name="velocity">
+                <param name="min">-10</param>
+                <param name="max">10</param>
+            </command_interface>
+            <state_interface name="velocity"/>
+            <state_interface name="position"/>
+        </joint>
+        <joint name="base_to_r_f_wheel">
+            <command_interface name="velocity">
+                <param name="min">-10</param>
+                <param name="max">10</param>
+            </command_interface>
+            <state_interface name="velocity"/>
+            <state_interface name="position"/>
+        </joint>
+        <joint name="base_to_r_m_wheel">
+            <command_interface name="velocity">
+                <param name="min">-10</param>
+                <param name="max">10</param>
+            </command_interface>
+            <state_interface name="velocity"/>
+            <state_interface name="position"/>
+        </joint>
+        <joint name="base_to_r_r_wheel">
+            <command_interface name="velocity">
+                <param name="min">-10</param>
+                <param name="max">10</param>
+            </command_interface>
+            <state_interface name="velocity"/>
+            <state_interface name="position"/>
+        </joint>
+    </ros2_control>
     <gazebo>
         <plugin name="gazebo_ros2_control" filename="libgazebo_ros2_control.so">
             <parameters>$(find rover_description)/config/my_controllers.yaml</parameters>
         </plugin>
-        <updateRate>20</updateRate>
+        <updateRate>30</updateRate>
  <!--   <ros>
           <remapping>odom:=odom/unfiltered</remapping>

File: rover_description/urdf/trk211.xacro (robot description, xacro)
@@ -3,5 +3,5 @@
   <!-- Включение файлов -->
   <xacro:include filename="chassis.xacro"/>
-  <xacro:include filename="gazebo_control.xacro"/>
+  <xacro:include filename="ros2_control.xacro"/>
   <xacro:include filename="imu.xacro"/>
   <xacro:include filename="$(find velodyne_description)/urdf/VLP-16.urdf.xacro"/>

Commit message: end of adding gazebo plugin

File: rover_description/urdf/ros2_control.xacro (robot description, xacro)
@@ -1,16 +1,10 @@
 <?xml version="1.0"?>
 <robot xmlns:xacro="http://www.ros.org/wiki/xacro" name="trk211">
+  <!-- Конфигурация ros2_control для Gazebo -->
   <ros2_control name="WheeledRobotSystem" type="system">
     <hardware>
-      <plugin>ros2_control_wheeled_robot_hardware/WheeledRobotHardware</plugin>
-      <!-- Параметры UDP-соединения -->
-      <param name="udp_ip">127.0.0.1</param>  <!-- IP робота  192.168.3.106, для отладки 127.0.0.1 -->
-      <param name="udp_port">8889</param>         <!-- Порт робота 4001, для отладки 8889 -->
-      <param name="local_port">8888</param>       <!-- Локальный порт 4001,  для отладки 8888 -->
-      <!-- Параметры колес -->
-      <param name="wheel_separation">0.8</param>  <!-- Расстояние между колесами (м) -->
-      <param name="wheel_radius">0.19</param>    <!-- Радиус колес (м) -->
-      <param name="send_timeout_ms">500</param>
-      <param name="receive_timeout_ms">500</param>
+      <plugin>gazebo_ros_control/GazeboWheeledRobotHardware</plugin>
+      <param name="wheel_separation">0.8</param>
+      <param name="wheel_radius">0.19</param>
     </hardware>
     <!-- Конфигурация суставов -->
@@ -46,73 +40,8 @@
     </joint>
   </ros2_control>
+  <!-- Конфигурация Gazebo -->
   <gazebo>
-    <plugin filename="ros2_control_wheeled_robot_hardware.so" name="ros2_control_wheeled_robot_hardware/WheeledRobotHardware">
-      <parameters>$(find rover_description)/config/my_controllers.yaml</parameters>
+    <plugin name="gazebo_ros_control" filename="libgazebo_ros_control.so">
     </plugin>
   </gazebo>
 </robot>
-<!--?xml version="1.0"?>
-<robot xmlns:xacro="http://www.ros.org/wiki/xacro">
-    <ros2_control name="GazeboSystem" type="system">
-        <hardware>
-            <plugin>gazebo_ros2_control/GazeboSystem</plugin>
-        </hardware>
-        <joint name="base_to_l_f_wheel">
-            <command_interface name="velocity">
-                <param name="min">-10</param>
-                <param name="max">10</param>
-            </command_interface>
-            <state_interface name="velocity"/>
-            <state_interface name="position"/>
-        </joint>
-        <joint name="base_to_l_m_wheel">
-            <command_interface name="velocity">
-                <param name="min">-10</param>
-                <param name="max">10</param>
-            </command_interface>
-            <state_interface name="velocity"/>
-            <state_interface name="position"/>
-        </joint>
-        <joint name="base_to_l_r_wheel">
-            <command_interface name="velocity">
-                <param name="min">-10</param>
-                <param name="max">10</param>
-            </command_interface>
-            <state_interface name="velocity"/>
-            <state_interface name="position"/>
-        </joint>
-        <joint name="base_to_r_f_wheel">
-            <command_interface name="velocity">
-                <param name="min">-10</param>
-                <param name="max">10</param>
-            </command_interface>
-            <state_interface name="velocity"/>
-            <state_interface name="position"/>
-        </joint>
-        <joint name="base_to_r_m_wheel">
-            <command_interface name="velocity">
-                <param name="min">-10</param>
-                <param name="max">10</param>
-            </command_interface>
-            <state_interface name="velocity"/>
-            <state_interface name="position"/>
-        </joint>
-        <joint name="base_to_r_r_wheel">
-            <command_interface name="velocity">
-                <param name="min">-10</param>
-                <param name="max">10</param>
-            </command_interface>
-            <state_interface name="velocity"/>
-            <state_interface name="position"/>
-        </joint>
-    </ros2_control>
-    <gazebo>
-        <plugin name="gazebo_ros2_control" filename="libgazebo_ros2_control.so">
-            <parameters>$(find rover_description)/config/my_controllers.yaml</parameters>
-        </plugin>
-        <updateRate>30</updateRate>
-        <<ros>
-          <remapping>odom:=odom/unfiltered</remapping>
-        </ros>>
-    </gazebo>
-</robot-->

Commit message: try to fix sim (((((

File: rover_description/urdf/ros2_control.xacro (robot description, xacro)
@@ -1,118 +1,43 @@
 <?xml version="1.0"?>
-<robot xmlns:xacro="http://www.ros.org/wiki/xacro" name="trk211">
-  <ros2_control name="WheeledRobotSystem" type="system">
+<robot xmlns:xacro="http://www.ros.org/wiki/xacro">
+  <ros2_control name="GazeboSystem" type="system">
     <hardware>
-      <plugin>ros2_control_wheeled_robot_hardware/WheeledRobotHardware</plugin>
-      <!-- Параметры UDP-соединения -->
-      <param name="udp_ip">127.0.0.1</param>  <!-- IP робота  192.168.3.106, для отладки 127.0.0.1 -->
-      <param name="udp_port">8889</param>         <!-- Порт робота 4001, для отладки 8889 -->
-      <param name="local_port">8888</param>       <!-- Локальный порт 4001,  для отладки 8888 -->
-      <!-- Параметры колес -->
-      <param name="wheel_separation">0.8</param>  <!-- Расстояние между колесами (м) -->
-      <param name="wheel_radius">0.19</param>    <!-- Радиус колес (м) -->
-      <param name="send_timeout_ms">500</param>
-      <param name="receive_timeout_ms">500</param>
+      <plugin>gazebo_ros2_control/GazeboSystem</plugin>
     </hardware>
-    <!-- Конфигурация суставов -->
     <joint name="base_to_left_forward_wheel">
+      <command_interface name="velocity"/>
       <state_interface name="velocity"/>
       <state_interface name="position"/>
-      <command_interface name="velocity"/>
     </joint>
     <joint name="base_to_left_middle_wheel">
+      <command_interface name="velocity"/>
       <state_interface name="velocity"/>
       <state_interface name="position"/>
-      <command_interface name="velocity"/>
     </joint>
     <joint name="base_to_left_rear_wheel">
+      <command_interface name="velocity"/>
       <state_interface name="velocity"/>
       <state_interface name="position"/>
-      <command_interface name="velocity"/>
     </joint>
     <joint name="base_to_right_forward_wheel">
+      <command_interface name="velocity"/>
       <state_interface name="velocity"/>
       <state_interface name="position"/>
-      <command_interface name="velocity"/>
     </joint>
     <joint name="base_to_right_middle_wheel">
+      <command_interface name="velocity"/>
       <state_interface name="velocity"/>
       <state_interface name="position"/>
-      <command_interface name="velocity"/>
     </joint>
     <joint name="base_to_right_rear_wheel">
+      <command_interface name="velocity"/>
       <state_interface name="velocity"/>
       <state_interface name="position"/>
-      <command_interface name="velocity"/>
     </joint>
   </ros2_control>
   <gazebo>
-    <plugin filename="ros2_control_wheeled_robot_hardware.so" name="ros2_control_wheeled_robot_hardware/WheeledRobotHardware">
+    <plugin name="gazebo_ros2_control" filename="libgazebo_ros2_control.so">
       <parameters>$(find rover_description)/config/my_controllers.yaml</parameters>
     </plugin>
   </gazebo>
 </robot>
-<!--?xml version="1.0"?>
-<robot xmlns:xacro="http://www.ros.org/wiki/xacro">
-    <ros2_control name="GazeboSystem" type="system">
-        <hardware>
-            <plugin>gazebo_ros2_control/GazeboSystem</plugin>
-        </hardware>
-        <joint name="base_to_l_f_wheel">
-            <command_interface name="velocity">
-                <param name="min">-10</param>
-                <param name="max">10</param>
-            </command_interface>
-            <state_interface name="velocity"/>
-            <state_interface name="position"/>
-        </joint>
-        <joint name="base_to_l_m_wheel">
-            <command_interface name="velocity">
-                <param name="min">-10</param>
-                <param name="max">10</param>
-            </command_interface>
-            <state_interface name="velocity"/>
-            <state_interface name="position"/>
-        </joint>
-        <joint name="base_to_l_r_wheel">
-            <command_interface name="velocity">
-                <param name="min">-10</param>
-                <param name="max">10</param>
-            </command_interface>
-            <state_interface name="velocity"/>
-            <state_interface name="position"/>
-        </joint>
-        <joint name="base_to_r_f_wheel">
-            <command_interface name="velocity">
-                <param name="min">-10</param>
-                <param name="max">10</param>
-            </command_interface>
-            <state_interface name="velocity"/>
-            <state_interface name="position"/>
-        </joint>
-        <joint name="base_to_r_m_wheel">
-            <command_interface name="velocity">
-                <param name="min">-10</param>
-                <param name="max">10</param>
-            </command_interface>
-            <state_interface name="velocity"/>
-            <state_interface name="position"/>
-        </joint>
-        <joint name="base_to_r_r_wheel">
-            <command_interface name="velocity">
-                <param name="min">-10</param>
-                <param name="max">10</param>
-            </command_interface>
-            <state_interface name="velocity"/>
-            <state_interface name="position"/>
-        </joint>
-    </ros2_control>
-    <gazebo>
-        <plugin name="gazebo_ros2_control" filename="libgazebo_ros2_control.so">
-            <parameters>$(find rover_description)/config/my_controllers.yaml</parameters>
-        </plugin>
-        <updateRate>30</updateRate>
-        <<ros>
-          <remapping>odom:=odom/unfiltered</remapping>
-        </ros>>
-    </gazebo>
-</robot-->
