Commit message: debug joy_params

File: rover_description/urdf/chassis.xacro (robot description, xacro)
@@ -194,5 +194,5 @@
   </xacro:macro>
   <xacro:wheel_joint
-    w_name="l_f"
+    w_name="left_forward"
     origin_y="${track/2}"
     origin_x="${wheelbase/2}"
@@ -202,5 +202,5 @@
     mu2="0.5"/>
   <xacro:wheel_joint
-    w_name="l_m"
+    w_name="left_middle"
     origin_y="${track/2}"
     origin_x="0"
@@ -210,5 +210,5 @@
     mu2="0.5"/>
   <xacro:wheel_joint
-    w_name="l_r"
+    w_name="left_rear"
     origin_y="${track/2}"
     origin_x="${-wheelbase/2}"
@@ -218,5 +218,5 @@
     mu2="0.5"/>
   <xacro:wheel_joint
-    w_name="r_f"
+    w_name="right_forward"
     origin_y="${-track/2}"
     origin_x="${wheelbase/2}"
@@ -226,5 +226,5 @@
     mu2="0.5"/>
   <xacro:wheel_joint
-    w_name="r_m"
+    w_name="right_middle"
     origin_y="${-track/2}"
     origin_x="0"
@@ -234,5 +234,5 @@
     mu2="0.5"/>
   <xacro:wheel_joint
-    w_name="r_r"
+    w_name="right_rear"
     origin_y="${-track/2}"
     origin_x="${-wheelbase/2}"

File: rover_description/urdf/gazebo_control.xacro (robot description, xacro)
@@ -1,3 +1,3 @@
-<?xml version="1.0"?>
+<!?xml version="1.0"?>
 <robot xmlns:xacro="http://www.ros.org/wiki/xacro">
     <gazebo>

File: rover_description/urdf/ros2_control.xacro (robot description, xacro)
@@ -1,3 +1,56 @@
 <?xml version="1.0"?>
+<robot xmlns:xacro="http://www.ros.org/wiki/xacro" name="trk211">
+  <ros2_control name="WheeledRobotSystem" type="system">
+    <hardware>
+      <plugin>ros2_control_wheeled_robot_hardware/WheeledRobotHardware</plugin>
+      <!-- Параметры UDP-соединения -->
+      <param name="udp_ip">127.0.0.1</param>  <!-- IP робота  192.168.3.106, для отладки 127.0.0.1 -->
+      <param name="udp_port">8889</param>         <!-- Порт робота 4001, для отладки 8889 -->
+      <param name="local_port">8888</param>       <!-- Локальный порт 4001,  для отладки 8888 -->
+      <!-- Параметры колес -->
+      <param name="wheel_separation">0.8</param>  <!-- Расстояние между колесами (м) -->
+      <param name="wheel_radius">0.19</param>    <!-- Радиус колес (м) -->
+      <param name="send_timeout_ms">500</param>
+      <param name="receive_timeout_ms">500</param>
+    </hardware>
+    <!-- Конфигурация суставов -->
+    <joint name="base_to_left_forward_wheel">
+      <state_interface name="velocity"/>
+      <state_interface name="position"/>
+      <command_interface name="velocity"/>
+    </joint>
+    <joint name="base_to_left_middle_wheel">
+      <state_interface name="velocity"/>
+      <state_interface name="position"/>
+      <command_interface name="velocity"/>
+    </joint>
+    <joint name="base_to_left_rear_wheel">
+      <state_interface name="velocity"/>
+      <state_interface name="position"/>
+      <command_interface name="velocity"/>
+    </joint>
+    <joint name="base_to_right_forward_wheel">
+      <state_interface name="velocity"/>
+      <state_interface name="position"/>
+      <command_interface name="velocity"/>
+    </joint>
+    <joint name="base_to_right_middle_wheel">
+      <state_interface name="velocity"/>
+      <state_interface name="position"/>
+      <command_interface name="velocity"/>
+    </joint>
+    <joint name="base_to_right_rear_wheel">
+      <state_interface name="velocity"/>
+      <state_interface name="position"/>
+      <command_interface name="velocity"/>
+    </joint>
+  </ros2_control>
+  <gazebo>
+    <plugin filename="ros2_control_wheeled_robot_hardware.so" name="ros2_control_wheeled_robot_hardware/WheeledRobotHardware">
+      <parameters>$(find rover_description)/config/my_controllers.yaml</parameters>
+    </plugin>
+  </gazebo>
+</robot>
+<!--?xml version="1.0"?>
 <robot xmlns:xacro="http://www.ros.org/wiki/xacro">
     <ros2_control name="GazeboSystem" type="system">
@@ -59,7 +112,7 @@
         </plugin>
         <updateRate>30</updateRate>
- <!--   <ros>
+        <<ros>
           <remapping>odom:=odom/unfiltered</remapping>
-        </ros> -->
+        </ros>>
     </gazebo>
-</robot>
+</robot-->

Commit message: fix simulation ros2_control, config.rviz that -> velodyne overload, added camera urdf logic and gazebo description

File: rover_description/urdf/chassis.xacro (robot description, xacro)
@@ -32,5 +32,5 @@
   <xacro:property name="visionbox_link_height" value="0.015" />
   <xacro:property name="wheel_mass" value="20.0" /><!-- please correct this -->
-  <xacro:property name="wheel_radius" value="0.19" /><!-- please correct this -->
+  <xacro:property name="wheel_radius" value="0.23" /><!-- please correct this -->
   <xacro:property name="wheel_height" value="0.15" /><!-- please correct this -->
   <xacro:property name="wheelbase" value="1.0" /><!-- please correct this -->
@@ -144,8 +144,5 @@
 		            ${ctrlbox_link_height/2+visionbox_link_height/2}" rpy="0 0 0"/>
   </joint>
-  <link name="front_camera_link"></link>
-  <!--xacro:sensor_d415 parent="front_camera_link" use_nominal_extrinsics="true" add_plug="false">
-    <origin xyz="0 0 0" rpy="0 0 0"/>
-  </xacro:sensor_d415-->
+  <link name="front_camera_link"/>
   <joint name="ctrlbox_to_camera_link" type="fixed">
     <parent link="ctrlbox_link"/>

File: rover_description/urdf/ros2_control.xacro (robot description, xacro)
@@ -5,5 +5,5 @@
             <plugin>gazebo_ros2_control/GazeboSystem</plugin>
         </hardware>
-        <joint name="base_to_l_f_wheel">
+        <joint name="base_to_left_forward_wheel">
             <command_interface name="velocity">
                 <param name="min">-10</param>
@@ -13,5 +13,5 @@
             <state_interface name="position"/>
         </joint>
-        <joint name="base_to_l_m_wheel">
+        <joint name="base_to_left_middle_wheel">
             <command_interface name="velocity">
                 <param name="min">-10</param>
@@ -21,5 +21,5 @@
             <state_interface name="position"/>
         </joint>
-        <joint name="base_to_l_r_wheel">
+        <joint name="base_to_left_rear_wheel">
             <command_interface name="velocity">
                 <param name="min">-10</param>
@@ -29,5 +29,5 @@
             <state_interface name="position"/>
         </joint>
-        <joint name="base_to_r_f_wheel">
+        <joint name="base_to_right_forward_wheel">
             <command_interface name="velocity">
                 <param name="min">-10</param>
@@ -37,5 +37,5 @@
             <state_interface name="position"/>
         </joint>
-        <joint name="base_to_r_m_wheel">
+        <joint name="base_to_right_middle_wheel">
             <command_interface name="velocity">
                 <param name="min">-10</param>
@@ -45,5 +45,5 @@
             <state_interface name="position"/>
         </joint>
-        <joint name="base_to_r_r_wheel">
+        <joint name="base_to_right_rear_wheel">
             <command_interface name="velocity">
                 <param name="min">-10</param>
@@ -57,7 +57,8 @@
         <plugin name="gazebo_ros2_control" filename="libgazebo_ros2_control.so">
             <parameters>$(find rover_description)/config/my_controllers.yaml</parameters>
+            <parameters>$(find rover_description)/config/gaz_ros2_ctl_use_sim.yaml</parameters>
         </plugin>
-        <updateRate>30</updateRate>
- <!--   <ros>
+        <!-- <updateRate>10</updateRate> -->
+        <!-- <ros>
           <remapping>odom:=odom/unfiltered</remapping>
         </ros> -->

File: rover_description/urdf/trk211.xacro (robot description, xacro)
@@ -3,5 +3,5 @@
   <!-- Включение файлов -->
   <xacro:include filename="chassis.xacro"/>
-  <xacro:include filename="imu.xacro"/>
+  <!-- <xacro:include filename="imu.xacro"/> -->
   <xacro:include filename="ros2_control.xacro"/>
   <xacro:include filename="$(find velodyne_description)/urdf/VLP-16.urdf.xacro"/>
@@ -22,10 +22,11 @@
                 <origin xyz="0 0 ${visionbox_link_height/2}" rpy="0 0 0" />
   </xacro:VLP-16>
-  <!--
   <xacro:include filename="$(find realsense2_description)/urdf/_d415.urdf.xacro"/>
+  <xacro:sensor_d415 parent="front_camera_link" use_nominal_extrinsics="true">
+    <origin xyz="0 0 0" rpy="0 0 0"/>
+  </xacro:sensor_d415>
   <xacro:include filename="depth_camera.xacro"/>
-  <xacro:include filename="gazebo_control.xacro"/>
+  <!--<xacro:include filename="gazebo_control.xacro"/>
   <xacro:include filename="ros2_control.xacro"/>
-  -->
-  <!--xacro:include filename="camera.xacro"/-->
+  <xacro:include filename="camera.xacro"/>-->
 </robot>

Commit message: ros2_control - trawelling work, localization slam problem

File: rover_description/urdf/chassis.xacro (robot description, xacro)
@@ -32,5 +32,5 @@
   <xacro:property name="visionbox_link_height" value="0.015" />
   <xacro:property name="wheel_mass" value="20.0" /><!-- please correct this -->
-  <xacro:property name="wheel_radius" value="0.23" /><!-- please correct this -->
+  <xacro:property name="wheel_radius" value="0.19" /><!-- please correct this -->
   <xacro:property name="wheel_height" value="0.15" /><!-- please correct this -->
   <xacro:property name="wheelbase" value="1.0" /><!-- please correct this -->
@@ -38,4 +38,6 @@
   <xacro:property name="clearance" value="0.2" />
   <xacro:property name="wheel_vertical_offset" value="0.03282"/>
+  <xacro:property name="mu1" value="0.2"/>
+  <xacro:property name="mu2" value="0.2"/>
   <xacro:arg name="laser_rotation" default="false"/>
   <link name="root_link">
@@ -150,5 +152,5 @@
     <origin xyz="${ctrlbox_link_length/2} 0.0 0.026" rpy="0 0 0"/>
   </joint>
-  <xacro:macro name="wheel_joint" params="w_name origin_x origin_y origin_z geometry_yaw mu1 mu2">
+  <xacro:macro name="wheel_joint" params="w_name origin_x origin_y origin_z geometry_yaw mu1=${mu1} mu2=${mu2}">
     <link name="${w_name}_wheel">
       <visual>
@@ -195,7 +197,5 @@
     origin_x="${wheelbase/2}"
     origin_z="${wheel_radius-base_link_height/2-clearance}"
-    geometry_yaw="0"
-    mu1="0.5"
-    mu2="0.5"/>
+    geometry_yaw="0"/>
   <xacro:wheel_joint
     w_name="left_middle"
@@ -203,7 +203,5 @@
     origin_x="0"
     origin_z="${wheel_radius-base_link_height/2-clearance}"
-    geometry_yaw="0"
-    mu1="0.5"
-    mu2="0.5"/>
+    geometry_yaw="0"/>
   <xacro:wheel_joint
     w_name="left_rear"
@@ -211,7 +209,5 @@
     origin_x="${-wheelbase/2}"
     origin_z="${wheel_radius-base_link_height/2-clearance}"
-    geometry_yaw="0"
-    mu1="0.5"
-    mu2="0.5"/>
+    geometry_yaw="0"/>
   <xacro:wheel_joint
     w_name="right_forward"
@@ -219,7 +215,5 @@
     origin_x="${wheelbase/2}"
     origin_z="${wheel_radius-base_link_height/2-clearance}"
-    geometry_yaw="${pi}"
-    mu1="0.5"
-    mu2="0.5"/>
+    geometry_yaw="${pi}"/>
   <xacro:wheel_joint
     w_name="right_middle"
@@ -227,7 +221,5 @@
     origin_x="0"
     origin_z="${wheel_radius-base_link_height/2-clearance}"
-    geometry_yaw="${pi}"
-    mu1="0.5"
-    mu2="0.5"/>
+    geometry_yaw="${pi}"/>
   <xacro:wheel_joint
     w_name="right_rear"
@@ -235,7 +227,5 @@
     origin_x="${-wheelbase/2}"
     origin_z="${wheel_radius-base_link_height/2-clearance}"
-    geometry_yaw="${pi}"
-    mu1="0.5"
-    mu2="0.5"/>
+    geometry_yaw="${pi}"/>
   <!-- GPS -->
   <link name="gps_link"></link>

Commit message: small updates, filter dropping message appears because of rviz

File: rover_description/urdf/chassis.xacro (robot description, xacro)
@@ -38,6 +38,6 @@
   <xacro:property name="clearance" value="0.2" />
   <xacro:property name="wheel_vertical_offset" value="0.03282"/>
-  <xacro:property name="mu1" value="0.2"/>
-  <xacro:property name="mu2" value="0.2"/>
+  <xacro:property name="mu1" value="0.5"/>
+  <xacro:property name="mu2" value="0.5"/>
   <xacro:arg name="laser_rotation" default="false"/>
   <link name="root_link">

Commit message: some fixes for ros2 control - still dismatching rotation in gz and rviz

File: rover_description/urdf/chassis.xacro (robot description, xacro)
@@ -32,12 +32,12 @@
   <xacro:property name="visionbox_link_height" value="0.015" />
   <xacro:property name="wheel_mass" value="20.0" /><!-- please correct this -->
-  <xacro:property name="wheel_radius" value="0.19" /><!-- please correct this -->
+  <xacro:property name="wheel_radius" value="0.23" /><!-- please correct this -->
   <xacro:property name="wheel_height" value="0.15" /><!-- please correct this -->
   <xacro:property name="wheelbase" value="1.0" /><!-- please correct this -->
-  <xacro:property name="track" value="0.8" />
+  <xacro:property name="track" value="0.9" />
   <xacro:property name="clearance" value="0.2" />
   <xacro:property name="wheel_vertical_offset" value="0.03282"/>
-  <xacro:property name="mu1" value="0.2"/>
-  <xacro:property name="mu2" value="0.2"/>
+  <xacro:property name="mu1" value="0.5"/>
+  <xacro:property name="mu2" value="0.5"/>
   <xacro:arg name="laser_rotation" default="false"/>
   <link name="root_link">

File: rover_description/urdf/ros2_control.xacro (robot description, xacro)
@@ -57,5 +57,4 @@
         <plugin name="gazebo_ros2_control" filename="libgazebo_ros2_control.so">
             <parameters>$(find rover_description)/config/my_controllers.yaml</parameters>
-            <parameters>$(find rover_description)/config/gaz_ros2_ctl_use_sim.yaml</parameters>
         </plugin>
         <!-- <updateRate>10</updateRate> -->
@@ -65,67 +64,2 @@
     </gazebo>
 </robot>
-<!--?xml version="1.0"?>
-<robot xmlns:xacro="http://www.ros.org/wiki/xacro">
-    <ros2_control name="GazeboSystem" type="system">
-        <hardware>
-            <plugin>gazebo_ros2_control/GazeboSystem</plugin>
-        </hardware>
-        <joint name="base_to_l_f_wheel">
-            <command_interface name="velocity">
-                <param name="min">-10</param>
-                <param name="max">10</param>
-            </command_interface>
-            <state_interface name="velocity"/>
-            <state_interface name="position"/>
-        </joint>
-        <joint name="base_to_l_m_wheel">
-            <command_interface name="velocity">
-                <param name="min">-10</param>
-                <param name="max">10</param>
-            </command_interface>
-            <state_interface name="velocity"/>
-            <state_interface name="position"/>
-        </joint>
-        <joint name="base_to_l_r_wheel">
-            <command_interface name="velocity">
-                <param name="min">-10</param>
-                <param name="max">10</param>
-            </command_interface>
-            <state_interface name="velocity"/>
-            <state_interface name="position"/>
-        </joint>
-        <joint name="base_to_r_f_wheel">
-            <command_interface name="velocity">
-                <param name="min">-10</param>
-                <param name="max">10</param>
-            </command_interface>
-            <state_interface name="velocity"/>
-            <state_interface name="position"/>
-        </joint>
-        <joint name="base_to_r_m_wheel">
-            <command_interface name="velocity">
-                <param name="min">-10</param>
-                <param name="max">10</param>
-            </command_interface>
-            <state_interface name="velocity"/>
-            <state_interface name="position"/>
-        </joint>
-        <joint name="base_to_r_r_wheel">
-            <command_interface name="velocity">
-                <param name="min">-10</param>
-                <param name="max">10</param>
-            </command_interface>
-            <state_interface name="velocity"/>
-            <state_interface name="position"/>
-        </joint>
-    </ros2_control>
-    <gazebo>
-        <plugin name="gazebo_ros2_control" filename="libgazebo_ros2_control.so">
-            <parameters>$(find rover_description)/config/my_controllers.yaml</parameters>
-        </plugin>
-        <updateRate>30</updateRate>
-        <<ros>
-          <remapping>odom:=odom/unfiltered</remapping>
-        </ros>>
-    </gazebo>
-</robot-->

File: rover_description/urdf/trk211.xacro (robot description, xacro)
@@ -14,5 +14,5 @@
                 samples="200"
                 collision_range="0.3"
-                min_range="0.9"
+                min_range="0.1"
                 max_range="5.0"
                 noise="0.0"

Commit message: run ekf_node

File: rover_description/urdf/chassis.xacro (robot description, xacro)
@@ -32,9 +32,9 @@
   <xacro:property name="visionbox_link_height" value="0.015" />
   <xacro:property name="wheel_mass" value="20.0" /><!-- please correct this -->
-  <xacro:property name="wheel_radius" value="0.19" /><!-- please correct this -->
-  <xacro:property name="wheel_height" value="0.15" /><!-- please correct this -->
+  <xacro:property name="wheel_radius" value="0.23" /><!-- please correct this -->
+  <xacro:property name="wheel_height" value="0.05" /><!-- please correct this -->
   <xacro:property name="wheelbase" value="1.0" /><!-- please correct this -->
-  <xacro:property name="track" value="0.8" />
-  <xacro:property name="clearance" value="0.2" />
+  <xacro:property name="track" value="0.9" />
+  <xacro:property name="clearance" value="0.25" />
   <xacro:property name="wheel_vertical_offset" value="0.03282"/>
   <xacro:property name="mu1" value="0.5"/>

File: rover_description/urdf/imu.xacro (robot description, xacro)
@@ -39,5 +39,5 @@
       <pose relative_to='xsens_link'>0 0 0 0 0 0</pose>
       <always_on>true</always_on>
-      <update_rate>100</update_rate>
+      <update_rate>50</update_rate>
       <!--reduced version of the plugin for ros2 without params-->
       <plugin filename="libgazebo_ros_imu_sensor.so" name="imu_plugin">

File: rover_description/urdf/trk211.xacro (robot description, xacro)
@@ -3,5 +3,5 @@
   <!-- Включение файлов -->
   <xacro:include filename="chassis.xacro"/>
-  <!-- <xacro:include filename="imu.xacro"/> -->
+  <xacro:include filename="imu.xacro"/>
   <xacro:include filename="ros2_control.xacro"/>
   <xacro:include filename="$(find velodyne_description)/urdf/VLP-16.urdf.xacro"/>
